Commit message: Meshcat visualized in drake

File: finger_description/urdf/powerhouse_finger.urdf (robot description, URDF)
Before this commit: robot powerhouse_finger, 5 links, 4 joints
Links:
- link base_link: geometry collision mesh filename=package://finger_description/meshes/collision/col_base_link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; visual mesh filename=package://finger_description/meshes/visual/base_link.obj
- link distal_phalanx: geometry collision mesh filename=package://finger_description/meshes/collision/col_distal_ph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; visual mesh filename=package://finger_description/meshes/visual/distal_phalanx.o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
- link mcp_link: geometry collision mesh filename=package://finger_description/meshes/collision/col_mcp_link.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; visual mesh filename=package://finger_description/meshes/visual/mcp_link.obj
- link middle_phalanx: geometry collision mesh filename=package://finger_description/meshes/collision/col_middle_ph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; visual mesh filename=package://finger_description/meshes/visual/middle_phalanx.o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
