Commit message: Add drake collision + contact params to URDF and blender export script

File: finger_description/urdf/powerhouse_finger_rviz.urdf.xacro (robot description, xacro)
@@ -1,16 +1,12 @@
 <?xml version="1.0"?>
-<robot name="powerhouse_finger" xmlns:xacro="http://www.ros.org/wiki/xacro" xmlns:drake="drake.mit.edu">
-  <!-- Generated by blender_export_drake.py from /home/jarmibe7/ws_rds/src/rds-powerhouse-software/finger_description/meshes/segment.blend -->
+<robot name="powerhouse_finger" xmlns:xacro="http://www.ros.org/wiki/xacro">
+  <!-- Generated by blender_export.py from /home/jarmibe7/ws_rds/src/rds-powerhouse-software/finger_description/meshes/segment.blend -->
   <!--
     mesh_ext: selects the mesh format for visual and collision geometry.
       stl  →  RViz  (default)
-      gltf →  Drake / Meshcat
+      gltf  →  Drake / Meshcat
     Usage:
       ros2 launch finger_description load_finger.launch.xml mesh_ext:=stl
       ros2 launch finger_sim finger_test_scene.launch.xml   mesh_ext:=gltf
-    Drake contact model:
-      Each <collision> carries <drake:proximity_properties> with
-      Hunt-Crossley parameters.  Adjacent links are filtered via
-      <drake:collision_filter_group> at the end of this file.
   -->
   <xacro:arg name="mesh_ext" default="gltf"/>
@@ -45,11 +41,4 @@
         <mesh filename="package://finger_description/meshes/collision/col_base_link.${ext}"/>
       </geometry>
-      <drake:proximity_properties>
-        <drake:compliant_hydroelastic/>
-        <drake:hydroelastic_modulus value="1e+07"/>
-        <drake:hunt_crossley_dissipation value="0.5"/>
-        <drake:mu_static value="0.8"/>
-        <drake:mu_dynamic value="0.6"/>
-      </drake:proximity_properties>
     </collision>
     <inertial>
@@ -79,11 +68,4 @@
         <mesh filename="package://finger_description/meshes/collision/col_mcp_link.${ext}"/>
       </geometry>
-      <drake:proximity_properties>
-        <drake:compliant_hydroelastic/>
-        <drake:hydroelastic_modulus value="1e+07"/>
-        <drake:hunt_crossley_dissipation value="0.5"/>
-        <drake:mu_static value="0.8"/>
-        <drake:mu_dynamic value="0.6"/>
-      </drake:proximity_properties>
     </collision>
     <inertial>
@@ -113,11 +95,4 @@
         <mesh filename="package://finger_description/meshes/collision/col_proximal_phalanx.${ext}"/>
       </geometry>
-      <drake:proximity_properties>
-        <drake:compliant_hydroelastic/>
-        <drake:hydroelastic_modulus value="1e+07"/>
-        <drake:hunt_crossley_dissipation value="0.5"/>
-        <drake:mu_static value="0.8"/>
-        <drake:mu_dynamic value="0.6"/>
-      </drake:proximity_properties>
     </collision>
     <inertial>
@@ -147,11 +122,4 @@
         <mesh filename="package://finger_description/meshes/collision/col_middle_phalanx.${ext}"/>
       </geometry>
-      <drake:proximity_properties>
-        <drake:compliant_hydroelastic/>
-        <drake:hydroelastic_modulus value="1e+07"/>
-        <drake:hunt_crossley_dissipation value="0.5"/>
-        <drake:mu_static value="0.8"/>
-        <drake:mu_dynamic value="0.6"/>
-      </drake:proximity_properties>
     </collision>
     <inertial>
@@ -181,11 +149,4 @@
         <mesh filename="package://finger_description/meshes/collision/col_distal_phalanx.${ext}"/>
       </geometry>
-      <drake:proximity_properties>
-        <drake:compliant_hydroelastic/>
-        <drake:hydroelastic_modulus value="5e+06"/>
-        <drake:hunt_crossley_dissipation value="1.0"/>
-        <drake:mu_static value="1.0"/>
-        <drake:mu_dynamic value="0.8"/>
-      </drake:proximity_properties>
     </collision>
     <inertial>
@@ -195,24 +156,3 @@
     </inertial>
   </link>
-  <!-- ═══ Drake collision filter groups ═══════════════════════════════ -->
-  <drake:collision_filter_group name="base_and_mcp">
-    <drake:member link="base_link"/>
-    <drake:member link="mcp_link"/>
-    <drake:ignored_collision_filter_group name="base_and_mcp"/>
-  </drake:collision_filter_group>
-  <drake:collision_filter_group name="mcp_and_proximal">
-    <drake:member link="mcp_link"/>
-    <drake:member link="proximal_phalanx"/>
-    <drake:ignored_collision_filter_group name="mcp_and_proximal"/>
-  </drake:collision_filter_group>
-  <drake:collision_filter_group name="proximal_and_middle">
-    <drake:member link="proximal_phalanx"/>
-    <drake:member link="middle_phalanx"/>
-    <drake:ignored_collision_filter_group name="proximal_and_middle"/>
-  </drake:collision_filter_group>
-  <drake:collision_filter_group name="middle_and_distal">
-    <drake:member link="middle_phalanx"/>
-    <drake:member link="distal_phalanx"/>
-    <drake:ignored_collision_filter_group name="middle_and_distal"/>
-  </drake:collision_filter_group>
 </robot>
