Commit message: Finish four bar linkage angle constraint

File: finger_description/urdf/powerhouse_finger.urdf.xacro (robot description, xacro)
@@ -127,5 +127,4 @@
     <limit lower="0.0" upper="1.57" effort="3.0" velocity="3.14"/>
     <dynamics damping="0.1" friction="0.05"/>
-    <mimic joint="pip_flexion" multiplier="0.85" offset="0.0"/>
   </joint>
   <!-- Distal phalanx -->

Commit message: New linkage URDF setup

File: finger_description/urdf/powerhouse_finger.urdf.xacro (robot description, xacro)
@@ -1,16 +1,16 @@
 <?xml version="1.0"?>
 <robot name="powerhouse_finger" xmlns:xacro="http://www.ros.org/wiki/xacro" xmlns:drake="drake.mit.edu">
-  <!-- Generated by blender_export_drake.py from /home/jarmibe7/ws_rds/src/rds-powerhouse-software/finger_description/meshes/segment.blend -->
+  <!-- Generated by blender_export_drake.py from /home/jarmibe7/ws_rds/src/rds-powerhouse-software/finger_description/meshes/segment_linkage.blend -->
   <!--
-    mesh_ext: selects the mesh format for visual and collision geometry.
-      stl  →  RViz  (default)
-      gltf →  Drake / Meshcat
-    Usage:
-      ros2 launch finger_description load_finger.launch.xml mesh_ext:=stl
-      ros2 launch finger_sim finger_test_scene.launch.xml   mesh_ext:=gltf
-    Drake contact model:
-      Each <collision> carries <drake:proximity_properties> with
-      Hunt-Crossley parameters.  Adjacent links are filtered via
-      <drake:collision_filter_group> at the end of this file.
+    mesh_ext: stl → RViz (default),  gltf → Drake/Meshcat
+    4-bar linkage:
+      left_bar / right_bar are visual-only passive links.
+      PIP-side pins → URDF revolute joints (left/right_bar_joint).
+      DIP-side pins → Drake AddFixedConstraint (NOT URDF joints).
+      dip_flexion has no mimic — driven by geometric loop closure.
+      Offsets are computed from joint_axes.yaml world_origin fields.
+    Drake contact:
+      Each <collision> carries <drake:proximity_properties>.
+      Adjacent links suppressed via <drake:collision_filter_group>.
   -->
   <xacro:arg name="mesh_ext" default="gltf"/>
@@ -99,8 +99,8 @@
     <origin xyz="0.013 0.0 -0.0006" rpy="0 0 0"/>
     <axis xyz="0.0 1.0 0.0"/>
-    <limit lower="0" upper="1.57" effort="5.0" velocity="3.14"/>
-    <dynamics damping="0.1" friction="0.05"/>
-  </joint>
-  <!-- Proximal phalanx -->
+    <limit lower="0.0" upper="1.57" effort="5.0" velocity="3.14"/>
+    <dynamics damping="0.1" friction="0.05"/>
+  </joint>
+  <!-- Proximal phalanx (ground link of 4-bar) -->
   <link name="proximal_phalanx">
     <visual>
@@ -131,10 +131,10 @@
     <parent link="proximal_phalanx"/>
     <child link="middle_phalanx"/>
-    <origin xyz="0.065 0.0 0.0004" rpy="0 0 0"/>
+    <origin xyz="0.065 0.0014 0.0004" rpy="0 0 0"/>
     <axis xyz="0.0 1.0 0.0"/>
     <limit lower="0.0" upper="1.57" effort="5.0" velocity="3.14"/>
     <dynamics damping="0.1" friction="0.05"/>
   </joint>
-  <!-- Middle phalanx -->
+  <!-- Middle phalanx — IS the coupler bar of the 4-bar linkage -->
   <link name="middle_phalanx">
     <visual>
@@ -165,10 +165,10 @@
     <parent link="middle_phalanx"/>
     <child link="distal_phalanx"/>
-    <origin xyz="0.04 0.0 0.0002" rpy="0 0 0"/>
+    <origin xyz="0.04 0.0019 0.0002" rpy="0 0 0"/>
     <axis xyz="0.0 1.0 0.0"/>
     <limit lower="0.0" upper="1.57" effort="3.0" velocity="3.14"/>
     <dynamics damping="0.1" friction="0.05"/>
   </joint>
-  <!-- Distal phalanx -->
+  <!-- Distal phalanx (driven link of 4-bar) -->
   <link name="distal_phalanx">
     <visual>
@@ -195,4 +195,49 @@
     </inertial>
   </link>
+  <!-- Left exterior bar — visual only, no collision, driven by loop closure -->
+  <link name="left_bar">
+    <visual>
+      <geometry>
+        <mesh filename="package://finger_description/meshes/visual/left_bar.${ext}"/>
+      </geometry>
+    </visual>
+    <inertial>
+      <mass value="0.001"/>
+      <origin xyz="0 0 0" rpy="0 0 0"/>
+      <inertia ixx="5e-07" ixy="0" ixz="0" iyy="5e-07" iyz="0" izz="5e-07"/>
+    </inertial>
+  </link>
+  <!-- Right exterior bar — visual only, no collision, driven by loop closure -->
+  <link name="right_bar">
+    <visual>
+      <geometry>
+        <mesh filename="package://finger_description/meshes/visual/right_bar.${ext}"/>
+      </geometry>
+    </visual>
+    <inertial>
+      <mass value="0.001"/>
+      <origin xyz="0 0 0" rpy="0 0 0"/>
+      <inertia ixx="5e-07" ixy="0" ixz="0" iyy="5e-07" iyz="0" izz="5e-07"/>
+    </inertial>
+  </link>
+  <!-- ═══ 4-bar exterior bar joints (branch off proximal_phalanx) ══ -->
+  <!-- Left Bar Joint -->
+  <joint name="left_bar_joint" type="revolute">
+    <parent link="proximal_phalanx"/>
+    <child link="left_bar"/>
+    <origin xyz="0.0613 0.0138 -0.0091" rpy="0 0 0"/>
+    <axis xyz="0.0 1.0 0.0"/>
+    <limit lower="0.0" upper="1.57" effort="0.0" velocity="3.14"/>
+    <dynamics damping="0.02" friction="0.01"/>
+  </joint>
+  <!-- Right Bar Joint -->
+  <joint name="right_bar_joint" type="revolute">
+    <parent link="proximal_phalanx"/>
+    <child link="right_bar"/>
+    <origin xyz="0.0618 -0.0121 -0.0091" rpy="0 0 0"/>
+    <axis xyz="0.0 1.0 0.0"/>
+    <limit lower="0.0" upper="1.57" effort="0.0" velocity="3.14"/>
+    <dynamics damping="0.02" friction="0.01"/>
+  </joint>
   <!-- ═══ Drake collision filter groups ═══════════════════════════════ -->
   <drake:collision_filter_group name="base_and_mcp">
@@ -216,3 +261,26 @@
     <drake:ignored_collision_filter_group name="middle_and_distal"/>
   </drake:collision_filter_group>
+  <drake:collision_filter_group name="proximal_and_bars">
+    <drake:member link="proximal_phalanx"/>
+    <drake:member link="left_bar"/>
+    <drake:member link="right_bar"/>
+    <drake:ignored_collision_filter_group name="proximal_and_bars"/>
+  </drake:collision_filter_group>
+  <drake:collision_filter_group name="bars_and_middle">
+    <drake:member link="left_bar"/>
+    <drake:member link="right_bar"/>
+    <drake:member link="middle_phalanx"/>
+    <drake:ignored_collision_filter_group name="bars_and_middle"/>
+  </drake:collision_filter_group>
+  <drake:collision_filter_group name="bars_and_distal">
+    <drake:member link="left_bar"/>
+    <drake:member link="right_bar"/>
+    <drake:member link="distal_phalanx"/>
+    <drake:ignored_collision_filter_group name="bars_and_distal"/>
+  </drake:collision_filter_group>
+  <drake:collision_filter_group name="bars_mutual">
+    <drake:member link="left_bar"/>
+    <drake:member link="right_bar"/>
+    <drake:ignored_collision_filter_group name="bars_mutual"/>
+  </drake:collision_filter_group>
 </robot>

Commit message: Fixing simulation bugs, adding diagram to sv

File: finger_description/urdf/powerhouse_finger.urdf.xacro (robot description, xacro)
@@ -55,5 +55,5 @@
     <inertial>
       <mass value="0.05"/>
-      <origin xyz="0 0 0" rpy="0 0 0"/>
+      <origin xyz="0.02038 -0.0 0.0975" rpy="0 0 0"/>
       <inertia ixx="1e-05" ixy="0" ixz="0" iyy="1e-05" iyz="0" izz="1e-05"/>
     </inertial>
@@ -66,5 +66,5 @@
     <axis xyz="0.0 0.0 1.0"/>
     <limit lower="-0.174533" upper="0.174533" effort="5.0" velocity="3.14"/>
-    <dynamics damping="0.1" friction="0.05"/>
+    <dynamics damping="0.0" friction="0.0"/>
   </joint>
   <!-- Space between MCP splay and flexion -->
@@ -89,5 +89,5 @@
     <inertial>
       <mass value="0.01"/>
-      <origin xyz="0 0 0" rpy="0 0 0"/>
+      <origin xyz="0.00073 0.00071 0.00014" rpy="0 0 0"/>
       <inertia ixx="1e-05" ixy="0" ixz="0" iyy="1e-05" iyz="0" izz="1e-05"/>
     </inertial>
@@ -100,5 +100,5 @@
     <axis xyz="0.0 1.0 0.0"/>
     <limit lower="0.0" upper="1.57" effort="5.0" velocity="3.14"/>
-    <dynamics damping="0.1" friction="0.05"/>
+    <dynamics damping="0.0" friction="0.001"/>
   </joint>
   <!-- Proximal phalanx (ground link of 4-bar) -->
@@ -123,5 +123,5 @@
     <inertial>
       <mass value="0.01"/>
-      <origin xyz="0 0 0" rpy="0 0 0"/>
+      <origin xyz="0.03712 0.00024 -0.0019" rpy="0 0 0"/>
       <inertia ixx="1e-05" ixy="0" ixz="0" iyy="1e-05" iyz="0" izz="1e-05"/>
     </inertial>
@@ -134,5 +134,5 @@
     <axis xyz="0.0 1.0 0.0"/>
     <limit lower="0.0" upper="1.57" effort="5.0" velocity="3.14"/>
-    <dynamics damping="0.1" friction="0.05"/>
+    <dynamics damping="0.0" friction="0.0"/>
   </joint>
   <!-- Middle phalanx — IS the coupler bar of the 4-bar linkage -->
@@ -157,5 +157,5 @@
     <inertial>
       <mass value="0.008"/>
-      <origin xyz="0 0 0" rpy="0 0 0"/>
+      <origin xyz="0.01223 0.00192 -0.00048" rpy="0 0 0"/>
       <inertia ixx="5e-06" ixy="0" ixz="0" iyy="5e-06" iyz="0" izz="5e-06"/>
     </inertial>
@@ -168,5 +168,5 @@
     <axis xyz="0.0 1.0 0.0"/>
     <limit lower="0.0" upper="1.57" effort="3.0" velocity="3.14"/>
-    <dynamics damping="0.1" friction="0.05"/>
+    <dynamics damping="0.0" friction="0.0"/>
   </joint>
   <!-- Distal phalanx (driven link of 4-bar) -->
@@ -191,5 +191,5 @@
     <inertial>
       <mass value="0.005"/>
-      <origin xyz="0 0 0" rpy="0 0 0"/>
+      <origin xyz="0.00948 -0.00161 0.00018" rpy="0 0 0"/>
       <inertia ixx="2e-06" ixy="0" ixz="0" iyy="2e-06" iyz="0" izz="2e-06"/>
     </inertial>
@@ -204,5 +204,5 @@
     <inertial>
       <mass value="0.001"/>
-      <origin xyz="0 0 0" rpy="0 0 0"/>
+      <origin xyz="0.01698 0.00021 0.00622" rpy="0 0 0"/>
       <inertia ixx="5e-07" ixy="0" ixz="0" iyy="5e-07" iyz="0" izz="5e-07"/>
     </inertial>
@@ -217,5 +217,5 @@
     <inertial>
       <mass value="0.001"/>
-      <origin xyz="0 0 0" rpy="0 0 0"/>
+      <origin xyz="0.01709 0.00017 0.00633" rpy="0 0 0"/>
       <inertia ixx="5e-07" ixy="0" ixz="0" iyy="5e-07" iyz="0" izz="5e-07"/>
     </inertial>
@@ -229,5 +229,5 @@
     <axis xyz="0.0 1.0 0.0"/>
     <limit lower="0.0" upper="1.57" effort="0.0" velocity="3.14"/>
-    <dynamics damping="0.02" friction="0.01"/>
+    <dynamics damping="0.0" friction="0.0"/>
   </joint>
   <!-- Right Bar Joint -->
@@ -238,5 +238,5 @@
     <axis xyz="0.0 1.0 0.0"/>
     <limit lower="0.0" upper="1.57" effort="0.0" velocity="3.14"/>
-    <dynamics damping="0.02" friction="0.01"/>
+    <dynamics damping="0.0" friction="0.0"/>
   </joint>
   <!-- ═══ Drake collision filter groups ═══════════════════════════════ -->
@@ -261,4 +261,9 @@
     <drake:ignored_collision_filter_group name="middle_and_distal"/>
   </drake:collision_filter_group>
+  <drake:collision_filter_group name="base_and_proximal">
+    <drake:member link="base_link"/>
+    <drake:member link="proximal_phalanx"/>
+    <drake:ignored_collision_filter_group name="base_and_proximal"/>
+  </drake:collision_filter_group>
   <drake:collision_filter_group name="proximal_and_bars">
     <drake:member link="proximal_phalanx"/>

Commit message: Fix linkage self collision

File: finger_description/urdf/powerhouse_finger.urdf.xacro (robot description, xacro)
@@ -1,5 +1,5 @@
 <?xml version="1.0"?>
 <robot name="powerhouse_finger" xmlns:xacro="http://www.ros.org/wiki/xacro" xmlns:drake="drake.mit.edu">
-  <!-- Generated by blender_export_drake.py from /home/jarmibe7/ws_rds/src/rds-powerhouse-software/finger_description/meshes/segment_linkage.blend -->
+  <!-- Generated by blender_export_drake.py from /home/jarmibe7/ws_rds/src/rds-powerhouse-software/finger_description/meshes/segment_simple_collision.blend -->
   <!--
     mesh_ext: stl → RViz (default),  gltf → Drake/Meshcat
@@ -190,7 +190,7 @@
     </collision>
     <inertial>
-      <mass value="0.005"/>
+      <mass value="0.5"/>
       <origin xyz="0.00948 -0.00161 0.00018" rpy="0 0 0"/>
-      <inertia ixx="2e-06" ixy="0" ixz="0" iyy="2e-06" iyz="0" izz="2e-06"/>
+      <inertia ixx="2e-05" ixy="0" ixz="0" iyy="2e-05" iyz="0" izz="2e-05"/>
     </inertial>
   </link>
@@ -203,7 +203,7 @@
     </visual>
     <inertial>
-      <mass value="0.001"/>
-      <origin xyz="0.01698 0.00021 0.00622" rpy="0 0 0"/>
-      <inertia ixx="5e-07" ixy="0" ixz="0" iyy="5e-07" iyz="0" izz="5e-07"/>
+      <mass value="0.1"/>
+      <origin xyz="0.0 0.0 0.0" rpy="0 0 0"/>
+      <inertia ixx="5e-05" ixy="0" ixz="0" iyy="5e-05" iyz="0" izz="5e-05"/>
     </inertial>
   </link>
@@ -216,7 +216,7 @@
     </visual>
     <inertial>
-      <mass value="0.001"/>
-      <origin xyz="0.01709 0.00017 0.00633" rpy="0 0 0"/>
-      <inertia ixx="5e-07" ixy="0" ixz="0" iyy="5e-07" iyz="0" izz="5e-07"/>
+      <mass value="0.1"/>
+      <origin xyz="0.01709 0.01322 0.00633" rpy="0 0 0"/>
+      <inertia ixx="5e-05" ixy="0" ixz="0" iyy="5e-05" iyz="0" izz="5e-05"/>
     </inertial>
   </link>
@@ -235,5 +235,5 @@
     <parent link="proximal_phalanx"/>
     <child link="right_bar"/>
-    <origin xyz="0.0618 -0.0121 -0.0091" rpy="0 0 0"/>
+    <origin xyz="0.0613 -0.0121 -0.0091" rpy="0 0 0"/>
     <axis xyz="0.0 1.0 0.0"/>
     <limit lower="0.0" upper="1.57" effort="0.0" velocity="3.14"/>

Commit message: Finger inertias, documentation

File: finger_description/urdf/powerhouse_finger.urdf.xacro (robot description, xacro)
@@ -54,7 +54,7 @@
     </collision>
     <inertial>
-      <mass value="0.05"/>
+      <mass value="0.183"/>
       <origin xyz="0.02038 -0.0 0.0975" rpy="0 0 0"/>
-      <inertia ixx="1e-05" ixy="0" ixz="0" iyy="1e-05" iyz="0" izz="1e-05"/>
+      <inertia ixx="0.0002589" ixy="0" ixz="0" iyy="0.0002239" iyz="0" izz="4.004e-05"/>
     </inertial>
   </link>
@@ -66,5 +66,5 @@
     <axis xyz="0.0 0.0 1.0"/>
     <limit lower="-0.174533" upper="0.174533" effort="5.0" velocity="3.14"/>
-    <dynamics damping="0.0" friction="0.0"/>
+    <dynamics damping="0.001" friction="0.0001"/>
   </joint>
   <!-- Space between MCP splay and flexion -->
@@ -88,7 +88,7 @@
     </collision>
     <inertial>
-      <mass value="0.01"/>
+      <mass value="0.04479276"/>
       <origin xyz="0.00073 0.00071 0.00014" rpy="0 0 0"/>
-      <inertia ixx="1e-05" ixy="0" ixz="0" iyy="1e-05" iyz="0" izz="1e-05"/>
+      <inertia ixx="8.781e-06" ixy="0" ixz="0" iyy="9.893e-06" iyz="0" izz="6.671e-06"/>
     </inertial>
   </link>
@@ -100,5 +100,5 @@
     <axis xyz="0.0 1.0 0.0"/>
     <limit lower="0.0" upper="1.57" effort="5.0" velocity="3.14"/>
-    <dynamics damping="0.0" friction="0.001"/>
+    <dynamics damping="0.001" friction="0.0001"/>
   </joint>
   <!-- Proximal phalanx (ground link of 4-bar) -->
@@ -122,7 +122,7 @@
     </collision>
     <inertial>
-      <mass value="0.01"/>
+      <mass value="0.072"/>
       <origin xyz="0.03712 0.00024 -0.0019" rpy="0 0 0"/>
-      <inertia ixx="1e-05" ixy="0" ixz="0" iyy="1e-05" iyz="0" izz="1e-05"/>
+      <inertia ixx="1.5e-05" ixy="0" ixz="0" iyy="4.649e-05" iyz="0" izz="4.385e-05"/>
     </inertial>
   </link>
@@ -134,5 +134,5 @@
     <axis xyz="0.0 1.0 0.0"/>
     <limit lower="0.0" upper="1.57" effort="5.0" velocity="3.14"/>
-    <dynamics damping="0.0" friction="0.0"/>
+    <dynamics damping="0.001" friction="0.0001"/>
   </joint>
   <!-- Middle phalanx — IS the coupler bar of the 4-bar linkage -->
@@ -156,5 +156,5 @@
     </collision>
     <inertial>
-      <mass value="0.008"/>
+      <mass value="0.01111115"/>
       <origin xyz="0.01223 0.00192 -0.00048" rpy="0 0 0"/>
       <inertia ixx="5e-06" ixy="0" ixz="0" iyy="5e-06" iyz="0" izz="5e-06"/>
@@ -168,5 +168,5 @@
     <axis xyz="0.0 1.0 0.0"/>
     <limit lower="0.0" upper="1.57" effort="3.0" velocity="3.14"/>
-    <dynamics damping="0.0" friction="0.0"/>
+    <dynamics damping="0.001" friction="0.0001"/>
   </joint>
   <!-- Distal phalanx (driven link of 4-bar) -->
@@ -190,7 +190,7 @@
     </collision>
     <inertial>
-      <mass value="0.5"/>
+      <mass value="0.03845096"/>
       <origin xyz="0.00948 -0.00161 0.00018" rpy="0 0 0"/>
-      <inertia ixx="2e-05" ixy="0" ixz="0" iyy="2e-05" iyz="0" izz="2e-05"/>
+      <inertia ixx="5.11e-06" ixy="0" ixz="0" iyy="7.503e-06" iyz="0" izz="7.527e-06"/>
     </inertial>
   </link>
@@ -203,7 +203,7 @@
     </visual>
     <inertial>
-      <mass value="0.1"/>
+      <mass value="0.00283571"/>
       <origin xyz="0.0 0.0 0.0" rpy="0 0 0"/>
-      <inertia ixx="5e-05" ixy="0" ixz="0" iyy="5e-05" iyz="0" izz="5e-05"/>
+      <inertia ixx="2.878e-08" ixy="0" ixz="0" iyy="3.747e-07" iyz="0" izz="3.53e-07"/>
     </inertial>
   </link>
@@ -216,7 +216,7 @@
     </visual>
     <inertial>
-      <mass value="0.1"/>
+      <mass value="0.00283571"/>
       <origin xyz="0.01709 0.01322 0.00633" rpy="0 0 0"/>
-      <inertia ixx="5e-05" ixy="0" ixz="0" iyy="5e-05" iyz="0" izz="5e-05"/>
+      <inertia ixx="2.878e-08" ixy="0" ixz="0" iyy="3.747e-07" iyz="0" izz="3.53e-07"/>
     </inertial>
   </link>
@@ -229,5 +229,5 @@
     <axis xyz="0.0 1.0 0.0"/>
     <limit lower="0.0" upper="1.57" effort="0.0" velocity="3.14"/>
-    <dynamics damping="0.0" friction="0.0"/>
+    <dynamics damping="0.001" friction="0.0001"/>
   </joint>
   <!-- Right Bar Joint -->
@@ -238,5 +238,5 @@
     <axis xyz="0.0 1.0 0.0"/>
     <limit lower="0.0" upper="1.57" effort="0.0" velocity="3.14"/>
-    <dynamics damping="0.0" friction="0.0"/>
+    <dynamics damping="0.001" friction="0.0001"/>
   </joint>
   <!-- ═══ Drake collision filter groups ═══════════════════════════════ -->

Commit message: Individual joint PD gains

File: finger_description/urdf/powerhouse_finger.urdf.xacro (robot description, xacro)
@@ -65,5 +65,5 @@
     <origin xyz="0.0195 -0.0 0.0983" rpy="0 0 0"/>
     <axis xyz="0.0 0.0 1.0"/>
-    <limit lower="-0.174533" upper="0.174533" effort="5.0" velocity="3.14"/>
+    <limit lower="-0.174533" upper="0.174533" effort="50.0" velocity="3.14"/>
     <dynamics damping="0.001" friction="0.0001"/>
   </joint>
@@ -99,5 +99,5 @@
     <origin xyz="0.013 0.0 -0.0006" rpy="0 0 0"/>
     <axis xyz="0.0 1.0 0.0"/>
-    <limit lower="0.0" upper="1.57" effort="5.0" velocity="3.14"/>
+    <limit lower="-0.785" upper="0.785" effort="50.0" velocity="3.14"/>
     <dynamics damping="0.001" friction="0.0001"/>
   </joint>
@@ -133,5 +133,5 @@
     <origin xyz="0.065 0.0014 0.0004" rpy="0 0 0"/>
     <axis xyz="0.0 1.0 0.0"/>
-    <limit lower="0.0" upper="1.57" effort="5.0" velocity="3.14"/>
+    <limit lower="0.0" upper="1.57" effort="50.0" velocity="3.14"/>
     <dynamics damping="0.001" friction="0.0001"/>
   </joint>
@@ -167,5 +167,5 @@
     <origin xyz="0.04 0.0019 0.0002" rpy="0 0 0"/>
     <axis xyz="0.0 1.0 0.0"/>
-    <limit lower="0.0" upper="1.57" effort="3.0" velocity="3.14"/>
+    <limit lower="0.0" upper="1.57" effort="50.0" velocity="3.14"/>
     <dynamics damping="0.001" friction="0.0001"/>
   </joint>
